Commit message: camera added

File: install/my_gesture_arm/share/my_gesture_arm/model/my_gesture_arm.xacro (robot description, xacro)
@@ -1,5 +1,5 @@
 <?xml version="1.0"?>
 <robot xmlns:xacro="http://ros.org/wiki/xacro" name="advanced_gesture_arm">
-<xacro:include filename="$(find my_gesture_arm)/model/gesture_arm.gazebo" />
+  <xacro:include filename="$(find my_gesture_arm)/model/gesture_arm.gazebo" />
   <xacro:property name="PI" value="3.14159"/>
   <xacro:macro name="cylinder_link" params="name radius length xyz rpy color mass">
@@ -114,5 +114,5 @@
     <origin xyz="0.225 0.275 0" rpy="0 0 0"/>
     <axis xyz="0 1 0"/>
-    <dynamics damping="0.1" friction="0.1"/>
+    <dynamics damping="0.5" friction="0.3"/>
   </joint>
   <!-- Front right wheel -->
@@ -123,5 +123,5 @@
     <origin xyz="0.225 -0.275 0" rpy="0 0 0"/>
     <axis xyz="0 1 0"/>
-    <dynamics damping="0.1" friction="0.1"/>
+    <dynamics damping="0.5" friction="0.3"/>
   </joint>
   <!-- Rear left wheel -->
@@ -132,5 +132,5 @@
     <origin xyz="-0.225 0.275 0" rpy="0 0 0"/>
     <axis xyz="0 1 0"/>
-    <dynamics damping="0.1" friction="0.1"/>
+    <dynamics damping="0.5" friction="0.3"/>
   </joint>
   <!-- Rear right wheel -->
@@ -141,5 +141,12 @@
     <origin xyz="-0.225 -0.275 0" rpy="0 0 0"/>
     <axis xyz="0 1 0"/>
-    <dynamics damping="0.1" friction="0.1"/>
+    <dynamics damping="0.5" friction="0.3"/>
+  </joint>
+  <!-- Camera link -->
+  <xacro:box_link name="camera_link" size="0.05 0.05 0.03" xyz="0 0 0.015" rpy="0 0 0" color="0.2 0.2 0.2 1.0" mass="0.1"/>
+  <joint name="camera_joint" type="fixed">
+    <parent link="base_link"/>
+    <child link="camera_link"/>
+    <origin xyz="0.3 0 0.1" rpy="0 0 0"/>
   </joint>
   <xacro:cylinder_link name="arm_mount" radius="0.08" length="0.4" xyz="0 0 0.2" rpy="0 0 0" color="0.4 0.4 0.4 1.0" mass="6.0"/>
@@ -155,5 +162,5 @@
     <axis xyz="0 0 1"/>
     <limit lower="-3.14" upper="3.14" effort="150.0" velocity="2.0"/>
-    <dynamics damping="5.0" friction="1.0"/>
+    <dynamics damping="10.0" friction="2.0"/>
   </joint>
   <xacro:cylinder_link name="shoulder_base" radius="0.07" length="0.08" xyz="0 0 0.04" rpy="0 0 0" color="0.7 0.0 0.0 1.0" mass="2.0"/>
@@ -164,5 +171,5 @@
     <axis xyz="0 1 0"/>
     <limit lower="-2.0" upper="2.0" effort="120.0" velocity="1.8"/>
-    <dynamics damping="5.0" friction="1.0"/>
+    <dynamics damping="8.0" friction="1.5"/>
   </joint>
   <xacro:cylinder_link name="upper_arm_link" radius="0.05" length="0.3" xyz="0 0 0.15" rpy="0 0 0" color="0.8 0.0 0.0 1.0" mass="1.5"/>
@@ -173,5 +180,5 @@
     <axis xyz="0 1 0"/>
     <limit lower="-2.5" upper="2.5" effort="80.0" velocity="2.0"/>
-    <dynamics damping="5.0" friction="1.0"/>
+    <dynamics damping="6.0" friction="1.0"/>
   </joint>
   <xacro:cylinder_link name="forearm_link" radius="0.045" length="0.25" xyz="0 0 0.125" rpy="0 0 0" color="0.0 1.0 0.0 1.0" mass="1.0"/>
@@ -182,5 +189,5 @@
     <axis xyz="1 0 0"/>
     <limit lower="-3.14" upper="3.14" effort="40.0" velocity="3.0"/>
-    <dynamics damping="5.0" friction="1.0"/>
+    <dynamics damping="4.0" friction="0.8"/>
   </joint>
   <xacro:cylinder_link name="wrist_roll_link" radius="0.04" length="0.06" xyz="0 0 0.03" rpy="0 0 0" color="0.0 0.8 0.8 1.0" mass="0.4"/>
@@ -191,5 +198,5 @@
     <axis xyz="0 1 0"/>
     <limit lower="-1.57" upper="1.57" effort="30.0" velocity="3.0"/>
-    <dynamics damping="5.0" friction="1.0"/>
+    <dynamics damping="3.0" friction="0.6"/>
   </joint>
   <xacro:cylinder_link name="wrist_pitch_link" radius="0.035" length="0.05" xyz="0 0 0.025" rpy="0 0 0" color="1.0 1.0 0.0 1.0" mass="0.3"/>
@@ -213,5 +220,5 @@
     <axis xyz="0 1 0"/>
     <limit lower="0.0" upper="0.03" effort="15.0" velocity="0.5"/>
-    <dynamics damping="0.01" friction="0.01"/>
+    <dynamics damping="0.1" friction="0.05"/>
   </joint>
   <xacro:box_link name="left_finger" size="0.03 0.01 0.06" xyz="0 0 0.03" rpy="0 0 0" color="1.0 0.5 0.0 1.0" mass="0.05"/>
@@ -223,12 +230,18 @@
     <axis xyz="0 -1 0"/>
     <limit lower="0.0" upper="0.03" effort="15.0" velocity="0.5"/>
-    <dynamics damping="0.01" friction="0.01"/>
+    <dynamics damping="0.1" friction="0.05"/>
     <mimic joint="left_finger_joint" multiplier="1" offset="0"/>
   </joint>
   <xacro:box_link name="right_finger" size="0.03 0.01 0.06" xyz="0 0 0.03" rpy="0 0 0" color="1.0 0.5 0.0 1.0" mass="0.05"/>
-    <!-- Gazebo ROS Control Plugin -->
+  <!-- State publisher -->
   <gazebo>
     <plugin name="gazebo_ros_control" filename="libgazebo_ros_control.so">
-      <robotNamespace>/gesture_arm</robotNamespace>
+      <robotNamespace>/advanced_gesture_arm</robotNamespace>
+    </plugin>
+    <plugin name="gazebo_ros_state" filename="libgazebo_ros_state.so">
+      <robotNamespace>/advanced_gesture_arm</robotNamespace>
+      <publish_rate>50</publish_rate>
+      <publish_tf>true</publish_tf>
+      <publish_joint_states>true</publish_joint_states>
     </plugin>
   </gazebo>

Commit message: camera added

File: install/my_gesture_arm/share/my_gesture_arm/model/my_gesture_arm.xacro (robot description, xacro)
@@ -1,6 +1,10 @@
 <?xml version="1.0"?>
-<robot xmlns:xacro="http://ros.org/wiki/xacro" name="advanced_gesture_arm">
+<robot xmlns:xacro="http://ros.org/wiki/xacro" name="my_gesture_arm">
+  <!-- Include the gazebo specific elements -->
   <xacro:include filename="$(find my_gesture_arm)/model/gesture_arm.gazebo" />
+  <!-- Constants -->
   <xacro:property name="PI" value="3.14159"/>
+  <xacro:property name="wheel_radius" value="0.1" />
+  <!-- Link and Joint Macros -->
   <xacro:macro name="cylinder_link" params="name radius length xyz rpy color mass">
     <link name="${name}">
@@ -53,17 +57,21 @@
         <origin xyz="${xyz}" rpy="${rpy}"/>
         <mass value="${mass}"/>
-        <xacro:property name="width" value="${size.split(' ')[0]}"/>
-        <xacro:property name="depth" value="${size.split(' ')[1]}"/>
-        <xacro:property name="height" value="${size.split(' ')[2]}"/>
         <inertia
-          ixx="${(1/12) * mass * (depth*depth + height*height)}"
+          ixx="${(1/12) * mass * (0.3*0.3 + 0.2*0.2)}"
           ixy="0.0"
           ixz="0.0"
-          iyy="${(1/12) * mass * (width*width + height*height)}"
+          iyy="${(1/12) * mass * (0.3*0.3 + 0.2*0.2)}"
           iyz="0.0"
-          izz="${(1/12) * mass * (width*width + depth*depth)}"/>
+          izz="${(1/12) * mass * (0.3*0.3 + 0.3*0.3)}"/>
       </inertial>
     </link>
   </xacro:macro>
+  <!-- Base Link -->
+  <link name="base_footprint"/>
+  <joint name="base_footprint_joint" type="fixed">
+    <parent link="base_footprint"/>
+    <child link="base_link"/>
+    <origin xyz="0 0 0.1" rpy="0 0 0"/>
+  </joint>
   <link name="base_link">
     <visual>
@@ -108,5 +116,5 @@
   </joint>
   <!-- Front left wheel -->
-  <xacro:cylinder_link name="front_left_wheel" radius="0.1" length="0.08" xyz="0 0 0" rpy="1.5708 0 0" color="0.0 0.0 0.0 1.0" mass="1.2"/>
+  <xacro:cylinder_link name="front_left_wheel" radius="${wheel_radius}" length="0.08" xyz="0 0 0" rpy="1.5708 0 0" color="0.0 0.0 0.0 1.0" mass="1.2"/>
   <joint name="front_left_wheel_joint" type="continuous">
     <parent link="wheel_mount_plate"/>
@@ -117,5 +125,5 @@
   </joint>
   <!-- Front right wheel -->
-  <xacro:cylinder_link name="front_right_wheel" radius="0.1" length="0.08" xyz="0 0 0" rpy="1.5708 0 0" color="0.0 0.0 0.0 1.0" mass="1.2"/>
+  <xacro:cylinder_link name="front_right_wheel" radius="${wheel_radius}" length="0.08" xyz="0 0 0" rpy="1.5708 0 0" color="0.0 0.0 0.0 1.0" mass="1.2"/>
   <joint name="front_right_wheel_joint" type="continuous">
     <parent link="wheel_mount_plate"/>
@@ -126,5 +134,5 @@
   </joint>
   <!-- Rear left wheel -->
-  <xacro:cylinder_link name="rear_left_wheel" radius="0.1" length="0.08" xyz="0 0 0" rpy="1.5708 0 0" color="0.0 0.0 0.0 1.0" mass="1.2"/>
+  <xacro:cylinder_link name="rear_left_wheel" radius="${wheel_radius}" length="0.08" xyz="0 0 0" rpy="1.5708 0 0" color="0.0 0.0 0.0 1.0" mass="1.2"/>
   <joint name="rear_left_wheel_joint" type="continuous">
     <parent link="wheel_mount_plate"/>
@@ -135,5 +143,5 @@
   </joint>
   <!-- Rear right wheel -->
-  <xacro:cylinder_link name="rear_right_wheel" radius="0.1" length="0.08" xyz="0 0 0" rpy="1.5708 0 0" color="0.0 0.0 0.0 1.0" mass="1.2"/>
+  <xacro:cylinder_link name="rear_right_wheel" radius="${wheel_radius}" length="0.08" xyz="0 0 0" rpy="1.5708 0 0" color="0.0 0.0 0.0 1.0" mass="1.2"/>
   <joint name="rear_right_wheel_joint" type="continuous">
     <parent link="wheel_mount_plate"/>
@@ -148,6 +156,20 @@
     <parent link="base_link"/>
     <child link="camera_link"/>
-    <origin xyz="0.3 0 0.1" rpy="0 0 0"/>
-  </joint>
+    <origin xyz="0.3 0 0.1" rpy="0 -0.2 0"/>
+  </joint>
+  <!-- Camera optical frame -->
+  <joint name="camera_optical_joint" type="fixed">
+    <parent link="camera_link"/>
+    <child link="camera_link_optical"/>
+    <origin xyz="0.0 0.0 0.0" rpy="${-PI/2} 0.0 ${-PI/2}"/>
+  </joint>
+  <link name="camera_link_optical">
+    <inertial>
+      <mass value="0.001"/>
+      <origin xyz="0 0 0" rpy="0 0 0"/>
+      <inertia ixx="0.0001" ixy="0" ixz="0" iyy="0.0001" iyz="0" izz="0.0001"/>
+    </inertial>
+  </link>
+  <!-- Robot Arm -->
   <xacro:cylinder_link name="arm_mount" radius="0.08" length="0.4" xyz="0 0 0.2" rpy="0 0 0" color="0.4 0.4 0.4 1.0" mass="6.0"/>
   <joint name="arm_mount_joint" type="fixed">
@@ -234,15 +256,3 @@
   </joint>
   <xacro:box_link name="right_finger" size="0.03 0.01 0.06" xyz="0 0 0.03" rpy="0 0 0" color="1.0 0.5 0.0 1.0" mass="0.05"/>
-  <!-- State publisher -->
-  <gazebo>
-    <plugin name="gazebo_ros_control" filename="libgazebo_ros_control.so">
-      <robotNamespace>/advanced_gesture_arm</robotNamespace>
-    </plugin>
-    <plugin name="gazebo_ros_state" filename="libgazebo_ros_state.so">
-      <robotNamespace>/advanced_gesture_arm</robotNamespace>
-      <publish_rate>50</publish_rate>
-      <publish_tf>true</publish_tf>
-      <publish_joint_states>true</publish_joint_states>
-    </plugin>
-  </gazebo>
 </robot>

Commit message: waste

File: install/my_gesture_arm/share/my_gesture_arm/model/my_gesture_arm.xacro (robot description, xacro)
@@ -122,5 +122,5 @@
     <origin xyz="0.225 0.275 0" rpy="0 0 0"/>
     <axis xyz="0 1 0"/>
-    <dynamics damping="0.5" friction="0.3"/>
+    <dynamics damping="0.1" friction="0.0"/>
   </joint>
   <!-- Front right wheel -->
@@ -131,5 +131,5 @@
     <origin xyz="0.225 -0.275 0" rpy="0 0 0"/>
     <axis xyz="0 1 0"/>
-    <dynamics damping="0.5" friction="0.3"/>
+    <dynamics damping="0.1" friction="0.0"/>
   </joint>
   <!-- Rear left wheel -->
@@ -140,5 +140,5 @@
     <origin xyz="-0.225 0.275 0" rpy="0 0 0"/>
     <axis xyz="0 1 0"/>
-    <dynamics damping="0.5" friction="0.3"/>
+    <dynamics damping="0.1" friction="0.0"/>
   </joint>
   <!-- Rear right wheel -->
@@ -149,5 +149,5 @@
     <origin xyz="-0.225 -0.275 0" rpy="0 0 0"/>
     <axis xyz="0 1 0"/>
-    <dynamics damping="0.5" friction="0.3"/>
+    <dynamics damping="0.1" friction="0.0"/>
   </joint>
   <!-- Camera link -->
@@ -184,5 +184,5 @@
     <axis xyz="0 0 1"/>
     <limit lower="-3.14" upper="3.14" effort="150.0" velocity="2.0"/>
-    <dynamics damping="10.0" friction="2.0"/>
+    <dynamics damping="5.0" friction="5.0"/>
   </joint>
   <xacro:cylinder_link name="shoulder_base" radius="0.07" length="0.08" xyz="0 0 0.04" rpy="0 0 0" color="0.7 0.0 0.0 1.0" mass="2.0"/>
@@ -193,5 +193,5 @@
     <axis xyz="0 1 0"/>
     <limit lower="-2.0" upper="2.0" effort="120.0" velocity="1.8"/>
-    <dynamics damping="8.0" friction="1.5"/>
+    <dynamics damping="5.0" friction="5.0"/>
   </joint>
   <xacro:cylinder_link name="upper_arm_link" radius="0.05" length="0.3" xyz="0 0 0.15" rpy="0 0 0" color="0.8 0.0 0.0 1.0" mass="1.5"/>
@@ -202,5 +202,5 @@
     <axis xyz="0 1 0"/>
     <limit lower="-2.5" upper="2.5" effort="80.0" velocity="2.0"/>
-    <dynamics damping="6.0" friction="1.0"/>
+    <dynamics damping="5.0" friction="5.0"/>
   </joint>
   <xacro:cylinder_link name="forearm_link" radius="0.045" length="0.25" xyz="0 0 0.125" rpy="0 0 0" color="0.0 1.0 0.0 1.0" mass="1.0"/>
@@ -211,5 +211,5 @@
     <axis xyz="1 0 0"/>
     <limit lower="-3.14" upper="3.14" effort="40.0" velocity="3.0"/>
-    <dynamics damping="4.0" friction="0.8"/>
+    <dynamics damping="5.0" friction="5.0"/>
   </joint>
   <xacro:cylinder_link name="wrist_roll_link" radius="0.04" length="0.06" xyz="0 0 0.03" rpy="0 0 0" color="0.0 0.8 0.8 1.0" mass="0.4"/>
@@ -220,5 +220,5 @@
     <axis xyz="0 1 0"/>
     <limit lower="-1.57" upper="1.57" effort="30.0" velocity="3.0"/>
-    <dynamics damping="3.0" friction="0.6"/>
+    <dynamics damping="5.0" friction="5.0"/>
   </joint>
   <xacro:cylinder_link name="wrist_pitch_link" radius="0.035" length="0.05" xyz="0 0 0.025" rpy="0 0 0" color="1.0 1.0 0.0 1.0" mass="0.3"/>

Commit message: teleop working

File: install/my_gesture_arm/share/my_gesture_arm/model/my_gesture_arm.xacro (robot description, xacro)
@@ -94,10 +94,10 @@
       <mass value="15.0"/>
       <inertia
-        ixx="0.6"
+        ixx="${(1/12) * 15.0 * (3*0.35*0.35 + 0.1*0.1)}"
         ixy="0.0"
         ixz="0.0"
-        iyy="0.6"
+        iyy="${(1/12) * 15.0 * (3*0.35*0.35 + 0.1*0.1)}"
         iyz="0.0"
-        izz="1.0"/>
+        izz="${0.5 * 15.0 * 0.35 * 0.35}"/>
     </inertial>
   </link>
@@ -120,7 +120,7 @@
     <parent link="wheel_mount_plate"/>
     <child link="front_left_wheel"/>
-    <origin xyz="0.225 0.275 0" rpy="0 0 0"/>
-    <axis xyz="0 1 0"/>
-    <dynamics damping="0.1" friction="0.0"/>
+    <origin xyz="0.225 0.275 -0.05" rpy="0 0 0"/>
+    <axis xyz="0 1 0"/>
+    <dynamics damping="0.1" friction="0.1"/>
   </joint>
   <!-- Front right wheel -->
@@ -129,7 +129,7 @@
     <parent link="wheel_mount_plate"/>
     <child link="front_right_wheel"/>
-    <origin xyz="0.225 -0.275 0" rpy="0 0 0"/>
-    <axis xyz="0 1 0"/>
-    <dynamics damping="0.1" friction="0.0"/>
+    <origin xyz="0.225 -0.275 -0.05" rpy="0 0 0"/>
+    <axis xyz="0 1 0"/>
+    <dynamics damping="0.1" friction="0.1"/>
   </joint>
   <!-- Rear left wheel -->
@@ -138,7 +138,7 @@
     <parent link="wheel_mount_plate"/>
     <child link="rear_left_wheel"/>
-    <origin xyz="-0.225 0.275 0" rpy="0 0 0"/>
-    <axis xyz="0 1 0"/>
-    <dynamics damping="0.1" friction="0.0"/>
+    <origin xyz="-0.225 0.275 -0.05" rpy="0 0 0"/>
+    <axis xyz="0 1 0"/>
+    <dynamics damping="0.1" friction="0.1"/>
   </joint>
   <!-- Rear right wheel -->
@@ -147,7 +147,14 @@
     <parent link="wheel_mount_plate"/>
     <child link="rear_right_wheel"/>
-    <origin xyz="-0.225 -0.275 0" rpy="0 0 0"/>
-    <axis xyz="0 1 0"/>
-    <dynamics damping="0.1" friction="0.0"/>
+    <origin xyz="-0.225 -0.275 -0.05" rpy="0 0 0"/>
+    <axis xyz="0 1 0"/>
+    <dynamics damping="0.1" friction="0.1"/>
+  </joint>
+  <!-- LIDAR Link -->
+  <xacro:box_link name="lidar_link" size="0.05 0.05 0.05" xyz="0 0 0.025" rpy="0 0 0" color="0.1 0.1 0.1 1.0" mass="0.1"/>
+  <joint name="lidar_joint" type="fixed">
+    <parent link="base_link"/>
+    <child link="lidar_link"/>
+    <origin xyz="0.3 0 0.15" rpy="0 0 0"/>
   </joint>
   <!-- Camera link -->
@@ -256,3 +263,51 @@
   </joint>
   <xacro:box_link name="right_finger" size="0.03 0.01 0.06" xyz="0 0 0.03" rpy="0 0 0" color="1.0 0.5 0.0 1.0" mass="0.05"/>
+  <!-- ROS2 Control Hardware Interface -->
+  <ros2_control name="GazeboSystem" type="system">
+    <hardware>
+      <plugin name="gazebo_ros2_control/GazeboSystem"/>
+    </hardware>
+    <joint name="shoulder_yaw_joint">
+      <command_interface name="position"/>
+      <state_interface name="position"/>
+      <state_interface name="velocity"/>
+      <state_interface name="effort"/>
+    </joint>
+    <joint name="shoulder_pitch_joint">
+      <command_interface name="position"/>
+      <state_interface name="position"/>
+      <state_interface name="velocity"/>
+      <state_interface name="effort"/>
+    </joint>
+    <joint name="elbow_joint">
+      <command_interface name="position"/>
+      <state_interface name="position"/>
+      <state_interface name="velocity"/>
+      <state_interface name="effort"/>
+    </joint>
+    <joint name="wrist_roll_joint">
+      <command_interface name="position"/>
+      <state_interface name="position"/>
+      <state_interface name="velocity"/>
+      <state_interface name="effort"/>
+    </joint>
+    <joint name="wrist_pitch_joint">
+      <command_interface name="position"/>
+      <state_interface name="position"/>
+      <state_interface name="velocity"/>
+      <state_interface name="effort"/>
+    </joint>
+    <joint name="left_finger_joint">
+      <command_interface name="position"/>
+      <state_interface name="position"/>
+      <state_interface name="velocity"/>
+      <state_interface name="effort"/>
+    </joint>
+    <joint name="right_finger_joint">
+      <command_interface name="position"/>
+      <state_interface name="position"/>
+      <state_interface name="velocity"/>
+      <state_interface name="effort"/>
+    </joint>
+  </ros2_control>
 </robot>

Commit message: added task world

File: install/my_gesture_arm/share/my_gesture_arm/model/my_gesture_arm.xacro (robot description, xacro)
@@ -1,6 +1,5 @@
 <?xml version="1.0"?>
 <robot xmlns:xacro="http://ros.org/wiki/xacro" name="my_gesture_arm">
-  <!-- Include the gazebo specific elements -->
-  <xacro:include filename="$(find my_gesture_arm)/model/gesture_arm.gazebo" />
+<xacro:include filename="$(find my_gesture_arm)/model/gesture_arm.gazebo" />
   <!-- Constants -->
   <xacro:property name="PI" value="3.14159"/>
@@ -190,6 +189,6 @@
     <origin xyz="0 0 0.4" rpy="0 0 0"/>
     <axis xyz="0 0 1"/>
-    <limit lower="-3.14" upper="3.14" effort="150.0" velocity="2.0"/>
-    <dynamics damping="5.0" friction="5.0"/>
+    <limit lower="-3.14" upper="3.14" effort="300.0" velocity="2.0"/>
+    <dynamics damping="0.5" friction="0.5"/>
   </joint>
   <xacro:cylinder_link name="shoulder_base" radius="0.07" length="0.08" xyz="0 0 0.04" rpy="0 0 0" color="0.7 0.0 0.0 1.0" mass="2.0"/>
@@ -199,6 +198,6 @@
     <origin xyz="0 0 0.08" rpy="0 0 0"/>
     <axis xyz="0 1 0"/>
-    <limit lower="-2.0" upper="2.0" effort="120.0" velocity="1.8"/>
-    <dynamics damping="5.0" friction="5.0"/>
+    <limit lower="-2.0" upper="2.0" effort="300.0" velocity="1.8"/>
+    <dynamics damping="0.5" friction="0.5"/>
   </joint>
   <xacro:cylinder_link name="upper_arm_link" radius="0.05" length="0.3" xyz="0 0 0.15" rpy="0 0 0" color="0.8 0.0 0.0 1.0" mass="1.5"/>
@@ -208,6 +207,6 @@
     <origin xyz="0 0 0.3" rpy="0 -0.2 0"/>
     <axis xyz="0 1 0"/>
-    <limit lower="-2.5" upper="2.5" effort="80.0" velocity="2.0"/>
-    <dynamics damping="5.0" friction="5.0"/>
+    <limit lower="-2.5" upper="2.5" effort="300.0" velocity="2.0"/>
+    <dynamics damping="0.5" friction="0.5"/>
   </joint>
   <xacro:cylinder_link name="forearm_link" radius="0.045" length="0.25" xyz="0 0 0.125" rpy="0 0 0" color="0.0 1.0 0.0 1.0" mass="1.0"/>
@@ -217,6 +216,6 @@
     <origin xyz="0 0 0.25" rpy="0 -0.1 0"/>
     <axis xyz="1 0 0"/>
-    <limit lower="-3.14" upper="3.14" effort="40.0" velocity="3.0"/>
-    <dynamics damping="5.0" friction="5.0"/>
+    <limit lower="-3.14" upper="3.14" effort="300.0" velocity="3.0"/>
+    <dynamics damping="0.5" friction="0.5"/>
   </joint>
   <xacro:cylinder_link name="wrist_roll_link" radius="0.04" length="0.06" xyz="0 0 0.03" rpy="0 0 0" color="0.0 0.8 0.8 1.0" mass="0.4"/>
@@ -226,6 +225,6 @@
     <origin xyz="0 0 0.06" rpy="0 0 0"/>
     <axis xyz="0 1 0"/>
-    <limit lower="-1.57" upper="1.57" effort="30.0" velocity="3.0"/>
-    <dynamics damping="5.0" friction="5.0"/>
+    <limit lower="-1.57" upper="1.57" effort="300.0" velocity="3.0"/>
+    <dynamics damping="0.5" friction="0.5"/>
   </joint>
   <xacro:cylinder_link name="wrist_pitch_link" radius="0.035" length="0.05" xyz="0 0 0.025" rpy="0 0 0" color="1.0 1.0 0.0 1.0" mass="0.3"/>
@@ -248,5 +247,5 @@
     <origin xyz="0.04 0.02 0.01" rpy="0 0 0"/>
     <axis xyz="0 1 0"/>
-    <limit lower="0.0" upper="0.03" effort="15.0" velocity="0.5"/>
+    <limit lower="0.0" upper="0.03" effort="50.0" velocity="0.5"/>
     <dynamics damping="0.1" friction="0.05"/>
   </joint>
@@ -258,5 +257,5 @@
     <origin xyz="0.04 -0.02 0.01" rpy="0 0 0"/>
     <axis xyz="0 -1 0"/>
-    <limit lower="0.0" upper="0.03" effort="15.0" velocity="0.5"/>
+    <limit lower="0.0" upper="0.03" effort="50.0" velocity="0.5"/>
     <dynamics damping="0.1" friction="0.05"/>
     <mimic joint="left_finger_joint" multiplier="1" offset="0"/>
