Commit message: dd_robot_with_imu

File: install/my_ddrobot/share/my_ddrobot/model/my_dd_robot_model.xacro (robot description, xacro)
@@ -1,159 +1 @@
-<?xml version="1.0"?>
-<robot xmlns:xacro = "http://www.ros.org/wiki/xacro" name="my_dd_robot">
-<xacro:property name="x_dim" value="0.6"/>
-<xacro:property name="y_dim" value="0.4"/>
-<xacro:property name="z_dim" value="0.2"/>
-<xacro:property name="robotname" value="my_dd"/>
-<xacro:property name= "wheel_radius" value = "0.1"/>
-<xacro:property name= "wheel_thickness" value = "0.05"/>
-<xacro:property name= "wheel_mass" value = "0.15"/>
-<xacro:macro name="inertial" params="mass">
-        <inertial>
-            <mass value="${mass}"/>
-            <inertia ixx="1e-3" ixy = "0.0" ixz="0.0" iyy="1e-3" iyz="0.0" izz="1e-3"/>
-            <origin xyz="0.0 0.0 0.0" rpy="0.0 0.0 0.0"/>
-        </inertial>
-</xacro:macro>
-<!--must be included only after defining xacro properties and macros-->
-<xacro:include filename="$(find my_ddrobot)/model/my_dd_robot.gazebo"/>
-    <material name="grey">
-        <color rgba="0.7 0.7 0.7 1" />
-    </material>
-    <material name="green">
-        <color rgba="0 0.6 0 1" />
-    </material>
-    <material name="white">
-        <color rgba="1 1 1 1"/>
-    </material>
-    <material name="yellow">
-        <color rgba="1 1 0 1"/>
-    </material>
-<!-- Base Footprint -->
-    <link name="base_footprint"/>
-<!-- Base link ; Body of the robot -->
-    <link name="base_link">
-        <visual>
-            <geometry>
-                <box size="${x_dim} ${y_dim} ${z_dim}" />
-            </geometry>
-            <origin xyz="0 0 0.1" rpy="0 0 0" />
-            <material name="green" />
-        </visual>
-<!-- Collision Geometry-->
-    <collision>
-        <geometry>
-            <box size="${x_dim} ${y_dim} ${z_dim}" />
-        </geometry>
-    </collision>
-<!-- Inertial Properties-->
-    <xacro:inertial mass="2"/>
-    </link>
-    <link name="left_wheel">
-        <visual>
-            <geometry>
-                <cylinder radius="${wheel_radius}" length="${wheel_thickness}"/>
-            </geometry>
-            <origin xyz="0 0 0" rpy="1.57 0 0" />
-            <material name="grey" />
-        </visual>
-        <collision>
-            <geometry>
-                <cylinder radius="${wheel_radius}" length="${wheel_thickness}"/>
-            </geometry>
-        </collision>
-        <xacro:inertial mass="${wheel_mass}"/>
-    </link>
-    <link name="right_wheel">
-        <visual>
-            <geometry>
-                <cylinder radius="${wheel_radius}" length="${wheel_thickness}"/>
-            </geometry>
-            <origin xyz="0 0 0" rpy="1.57 0 0" />
-            <material name="grey" />
-        </visual>
-        <collision>
-            <geometry>
-                <cylinder radius="${wheel_radius}" length="${wheel_thickness}"/>
-            </geometry>
-        </collision>
-     <xacro:inertial mass="${wheel_mass}"/>
-    </link>
-    <link name="caster_wheel">
-        <visual>
-            <geometry>
-                <sphere radius="0.05"/>
-            </geometry>
-            <origin xyz="0 0 0" rpy="0 0 0" />
-            <material name="grey" />
-        </visual>
-        <inertial>
-            <mass value="${wheel_mass}"/>
-            <inertia ixx="1e-3" ixy = "0.0" ixz="0.0" iyy="1e-3" iyz="0.0" izz="1e-3"/>
-        </inertial>
-    </link>
-<!-- +++++++++++++++ Camera Link  ++++++++++++++++++-->
-    <link name="camera_link">
-        <visual>
-             <geometry>
-                <box size="0.05 0.05 0.05"/>
-            </geometry>
-                <origin xyz="0 0 0" rpy="0 0 0" />
-            <material name="yellow" />
-        </visual>
-<!-- Collision Geometry-->
-    <collision>
-        <geometry>
-            <box size="0.05 0.05 0.05" />
-        </geometry>
-    </collision>
-<!-- Inertial Properties-->
-    <xacro:inertial mass="0.2"/>
-    </link>
-<!-- Body to Base Joint-->
-    <joint name="base_joint" type="fixed">
-        <parent link="base_footprint"/>
-        <child link="base_link"/>
-        <origin xyz="0 0 0.1" rpy="0 0 0"/>
-    </joint>
-<!--___________________________________________________________-->
-<!--Left wheel to Body Joint-->
-    <joint name="base_left_wheel_joint" type="continuous">
-        <parent link="base_link"/>
-        <child link="left_wheel"/>
-        <origin xyz="-0.15 0.225 0" rpy="0 0 0"/>
-        <axis xyz="0 1 0"/>
-<!--Wheel Dynamics -->
-        <dynamics damping = "1.0" friction ="0.4"/>
-    </joint>
-<!--___________________________________________________________-->
-<!--Left wheel to Body Joint-->
-    <joint name="base_right_wheel_joint" type="continuous">
-        <parent link="base_link"/>
-        <child link="right_wheel"/>
-        <origin xyz="-0.15 -0.225 0" rpy="0 0 0"/>
-        <axis xyz="0 1 0"/>
-<!--Wheel Dynamics -->
-        <dynamics damping = "1.0" friction ="0.4"/>
-    </joint>
-<!--___________________________________________________________-->
-<!--Caster Wheel to Body Joint-->
-    <joint name="base_caster_wheel_joint" type="fixed">
-        <parent link="base_link"/>
-        <child link="caster_wheel"/>
-        <origin xyz="0.2 0 -0.05" rpy="0 0 0"/>
-    </joint>
-<!--___________________________________________________________-->
-<!--Camera to Body Joint -->
-      <joint name="base_camera_joint" type="fixed">
-        <parent link="base_link"/>
-        <child link="camera_link"/>
-        <origin xyz="${x_dim/2 - 0.05/2} 0 ${z_dim+ (0.05/2)}" rpy="0 0 0"/>
-    </joint>
-<!--___________________________________________________________-->
-<!-- Camera Joint
-<joint name="camera_optical_joint" type="fixed">
-    <parent link="camera_link"/>
-    <child link="child_link_optical"/>
-    <origin xyz="0.0 0.0 0.0" rpy="0.0 0.0 0.0"/>
-</joint>-->
-</robot>
+/home/aniketh05/ros2_ws/src/my_ddrobot/model/my_dd_robot_model.xacro

File: install/my_gesture_arm/share/my_gesture_arm/model/my_gesture_arm.xacro (robot description, xacro)
@@ -1,312 +1 @@
-<?xml version="1.0"?>
-<robot xmlns:xacro="http://ros.org/wiki/xacro" name="my_gesture_arm">
-<xacro:include filename="$(find my_gesture_arm)/model/gesture_arm.gazebo" />
-  <!-- Constants -->
-  <xacro:property name="PI" value="3.14159"/>
-  <xacro:property name="wheel_radius" value="0.1" />
-  <!-- Link and Joint Macros -->
-  <xacro:macro name="cylinder_link" params="name radius length xyz rpy color mass">
-    <link name="${name}">
-      <visual>
-        <origin xyz="${xyz}" rpy="${rpy}"/>
-        <geometry>
-          <cylinder radius="${radius}" length="${length}"/>
-        </geometry>
-        <material name="">
-          <color rgba="${color}"/>
-        </material>
-      </visual>
-      <collision>
-        <origin xyz="${xyz}" rpy="${rpy}"/>
-        <geometry>
-          <cylinder radius="${radius}" length="${length}"/>
-        </geometry>
-      </collision>
-      <inertial>
-        <origin xyz="${xyz}" rpy="${rpy}"/>
-        <mass value="${mass}"/>
-        <inertia
-          ixx="${(1/12) * mass * (3*radius*radius + length*length)}"
-          ixy="0.0"
-          ixz="0.0"
-          iyy="${(1/12) * mass * (3*radius*radius + length*length)}"
-          iyz="0.0"
-          izz="${0.5 * mass * radius * radius}"/>
-      </inertial>
-    </link>
-  </xacro:macro>
-  <xacro:macro name="box_link" params="name size xyz rpy color mass">
-    <link name="${name}">
-      <visual>
-        <origin xyz="${xyz}" rpy="${rpy}"/>
-        <geometry>
-          <box size="${size}"/>
-        </geometry>
-        <material name="">
-          <color rgba="${color}"/>
-        </material>
-      </visual>
-      <collision>
-        <origin xyz="${xyz}" rpy="${rpy}"/>
-        <geometry>
-          <box size="${size}"/>
-        </geometry>
-      </collision>
-      <inertial>
-        <origin xyz="${xyz}" rpy="${rpy}"/>
-        <mass value="${mass}"/>
-        <inertia
-          ixx="${(1/12) * mass * (0.3*0.3 + 0.2*0.2)}"
-          ixy="0.0"
-          ixz="0.0"
-          iyy="${(1/12) * mass * (0.3*0.3 + 0.2*0.2)}"
-          iyz="0.0"
-          izz="${(1/12) * mass * (0.3*0.3 + 0.3*0.3)}"/>
-      </inertial>
-    </link>
-  </xacro:macro>
-  <!-- Base Link -->
-  <link name="base_footprint"/>
-  <joint name="base_footprint_joint" type="fixed">
-    <parent link="base_footprint"/>
-    <child link="base_link"/>
-    <origin xyz="0 0 0.1" rpy="0 0 0"/>
-  </joint>
-  <link name="base_link">
-    <visual>
-      <origin xyz="0 0 0.05" rpy="0 0 0"/>
-      <geometry>
-        <cylinder radius="0.35" length="0.1"/>
-      </geometry>
-      <material name="">
-        <color rgba="0.0 0.0 1.0 1.0"/>
-      </material>
-    </visual>
-    <collision>
-      <origin xyz="0 0 0.05" rpy="0 0 0"/>
-      <geometry>
-        <cylinder radius="0.35" length="0.1"/>
-      </geometry>
-    </collision>
-    <inertial>
-      <origin xyz="0 0 0.05" rpy="0 0 0"/>
-      <mass value="15.0"/>
-      <inertia
-        ixx="${(1/12) * 15.0 * (3*0.35*0.35 + 0.1*0.1)}"
-        ixy="0.0"
-        ixz="0.0"
-        iyy="${(1/12) * 15.0 * (3*0.35*0.35 + 0.1*0.1)}"
-        iyz="0.0"
-        izz="${0.5 * 15.0 * 0.35 * 0.35}"/>
-    </inertial>
-  </link>
-  <!-- Chassis -->
-  <xacro:box_link name="chassis_base" size="0.65 0.5 0.08" xyz="0 0 0.04" rpy="0 0 0" color="0.3 0.3 0.3 1.0" mass="10.0"/>
-  <joint name="chassis_joint" type="fixed">
-    <parent link="base_link"/>
-    <child link="chassis_base"/>
-    <origin xyz="0 0 0" rpy="0 0 0"/>
-  </joint>
-  <xacro:box_link name="wheel_mount_plate" size="0.55 0.6 0.05" xyz="0 0 0.025" rpy="0 0 0" color="0.2 0.2 0.2 1.0" mass="5.0"/>
-  <joint name="wheel_mount_joint" type="fixed">
-    <parent link="base_link"/>
-    <child link="wheel_mount_plate"/>
-    <origin xyz="0 0 -0.05" rpy="0 0 0"/>
-  </joint>
-  <!-- Front left wheel -->
-  <xacro:cylinder_link name="front_left_wheel" radius="${wheel_radius}" length="0.08" xyz="0 0 0" rpy="1.5708 0 0" color="0.0 0.0 0.0 1.0" mass="1.2"/>
-  <joint name="front_left_wheel_joint" type="continuous">
-    <parent link="wheel_mount_plate"/>
-    <child link="front_left_wheel"/>
-    <origin xyz="0.225 0.275 -0.05" rpy="0 0 0"/>
-    <axis xyz="0 1 0"/>
-    <dynamics damping="0.1" friction="0.1"/>
-  </joint>
-  <!-- Front right wheel -->
-  <xacro:cylinder_link name="front_right_wheel" radius="${wheel_radius}" length="0.08" xyz="0 0 0" rpy="1.5708 0 0" color="0.0 0.0 0.0 1.0" mass="1.2"/>
-  <joint name="front_right_wheel_joint" type="continuous">
-    <parent link="wheel_mount_plate"/>
-    <child link="front_right_wheel"/>
-    <origin xyz="0.225 -0.275 -0.05" rpy="0 0 0"/>
-    <axis xyz="0 1 0"/>
-    <dynamics damping="0.1" friction="0.1"/>
-  </joint>
-  <!-- Rear left wheel -->
-  <xacro:cylinder_link name="rear_left_wheel" radius="${wheel_radius}" length="0.08" xyz="0 0 0" rpy="1.5708 0 0" color="0.0 0.0 0.0 1.0" mass="1.2"/>
-  <joint name="rear_left_wheel_joint" type="continuous">
-    <parent link="wheel_mount_plate"/>
-    <child link="rear_left_wheel"/>
-    <origin xyz="-0.225 0.275 -0.05" rpy="0 0 0"/>
-    <axis xyz="0 1 0"/>
-    <dynamics damping="0.1" friction="0.1"/>
-  </joint>
-  <!-- Rear right wheel -->
-  <xacro:cylinder_link name="rear_right_wheel" radius="${wheel_radius}" length="0.08" xyz="0 0 0" rpy="1.5708 0 0" color="0.0 0.0 0.0 1.0" mass="1.2"/>
-  <joint name="rear_right_wheel_joint" type="continuous">
-    <parent link="wheel_mount_plate"/>
-    <child link="rear_right_wheel"/>
-    <origin xyz="-0.225 -0.275 -0.05" rpy="0 0 0"/>
-    <axis xyz="0 1 0"/>
-    <dynamics damping="0.1" friction="0.1"/>
-  </joint>
-  <!-- LIDAR Link -->
-  <xacro:box_link name="lidar_link" size="0.05 0.05 0.05" xyz="0 0 0.025" rpy="0 0 0" color="0.1 0.1 0.1 1.0" mass="0.1"/>
-  <joint name="lidar_joint" type="fixed">
-    <parent link="base_link"/>
-    <child link="lidar_link"/>
-    <origin xyz="0.3 0 0.15" rpy="0 0 0"/>
-  </joint>
-  <!-- Camera link -->
-  <xacro:box_link name="camera_link" size="0.05 0.05 0.03" xyz="0 0 0.015" rpy="0 0 0" color="0.2 0.2 0.2 1.0" mass="0.1"/>
-  <joint name="camera_joint" type="fixed">
-    <parent link="base_link"/>
-    <child link="camera_link"/>
-    <origin xyz="0.3 0 0.1" rpy="0 -0.2 0"/>
-  </joint>
-  <!-- Camera optical frame -->
-  <joint name="camera_optical_joint" type="fixed">
-    <parent link="camera_link"/>
-    <child link="camera_link_optical"/>
-    <origin xyz="0.0 0.0 0.0" rpy="${-PI/2} 0.0 ${-PI/2}"/>
-  </joint>
-  <link name="camera_link_optical">
-    <inertial>
-      <mass value="0.001"/>
-      <origin xyz="0 0 0" rpy="0 0 0"/>
-      <inertia ixx="0.0001" ixy="0" ixz="0" iyy="0.0001" iyz="0" izz="0.0001"/>
-    </inertial>
-  </link>
-  <!-- Robot Arm -->
-  <xacro:cylinder_link name="arm_mount" radius="0.08" length="0.4" xyz="0 0 0.2" rpy="0 0 0" color="0.4 0.4 0.4 1.0" mass="6.0"/>
-  <joint name="arm_mount_joint" type="fixed">
-    <parent link="base_link"/>
-    <child link="arm_mount"/>
-    <origin xyz="0 0 0.1" rpy="0 0 0"/>
-  </joint>
-  <joint name="shoulder_yaw_joint" type="revolute">
-    <parent link="arm_mount"/>
-    <child link="shoulder_base"/>
-    <origin xyz="0 0 0.4" rpy="0 0 0"/>
-    <axis xyz="0 0 1"/>
-    <limit lower="-3.14" upper="3.14" effort="300.0" velocity="2.0"/>
-    <dynamics damping="0.5" friction="0.5"/>
-  </joint>
-  <xacro:cylinder_link name="shoulder_base" radius="0.07" length="0.08" xyz="0 0 0.04" rpy="0 0 0" color="0.7 0.0 0.0 1.0" mass="2.0"/>
-  <joint name="shoulder_pitch_joint" type="revolute">
-    <parent link="shoulder_base"/>
-    <child link="upper_arm_link"/>
-    <origin xyz="0 0 0.08" rpy="0 0 0"/>
-    <axis xyz="0 1 0"/>
-    <limit lower="-2.0" upper="2.0" effort="300.0" velocity="1.8"/>
-    <dynamics damping="0.5" friction="0.5"/>
-  </joint>
-  <xacro:cylinder_link name="upper_arm_link" radius="0.05" length="0.3" xyz="0 0 0.15" rpy="0 0 0" color="0.8 0.0 0.0 1.0" mass="1.5"/>
-  <joint name="elbow_joint" type="revolute">
-    <parent link="upper_arm_link"/>
-    <child link="forearm_link"/>
-    <origin xyz="0 0 0.3" rpy="0 -0.2 0"/>
-    <axis xyz="0 1 0"/>
-    <limit lower="-2.5" upper="2.5" effort="300.0" velocity="2.0"/>
-    <dynamics damping="0.5" friction="0.5"/>
-  </joint>
-  <xacro:cylinder_link name="forearm_link" radius="0.045" length="0.25" xyz="0 0 0.125" rpy="0 0 0" color="0.0 1.0 0.0 1.0" mass="1.0"/>
-  <joint name="wrist_roll_joint" type="revolute">
-    <parent link="forearm_link"/>
-    <child link="wrist_roll_link"/>
-    <origin xyz="0 0 0.25" rpy="0 -0.1 0"/>
-    <axis xyz="1 0 0"/>
-    <limit lower="-3.14" upper="3.14" effort="300.0" velocity="3.0"/>
-    <dynamics damping="0.5" friction="0.5"/>
-  </joint>
-  <xacro:cylinder_link name="wrist_roll_link" radius="0.04" length="0.06" xyz="0 0 0.03" rpy="0 0 0" color="0.0 0.8 0.8 1.0" mass="0.4"/>
-  <joint name="wrist_pitch_joint" type="revolute">
-    <parent link="wrist_roll_link"/>
-    <child link="wrist_pitch_link"/>
-    <origin xyz="0 0 0.06" rpy="0 0 0"/>
-    <axis xyz="0 1 0"/>
-    <limit lower="-1.57" upper="1.57" effort="300.0" velocity="3.0"/>
-    <dynamics damping="0.5" friction="0.5"/>
-  </joint>
-  <xacro:cylinder_link name="wrist_pitch_link" radius="0.035" length="0.05" xyz="0 0 0.025" rpy="0 0 0" color="1.0 1.0 0.0 1.0" mass="0.3"/>
-  <joint name="end_effector_joint" type="fixed">
-    <parent link="wrist_pitch_link"/>
-    <child link="end_effector"/>
-    <origin xyz="0 0 0.05" rpy="0 -0.1 0"/>
-  </joint>
-  <xacro:cylinder_link name="end_effector" radius="0.03" length="0.02" xyz="0 0 0.01" rpy="0 0 0" color="0.0 0.0 0.0 1.0" mass="0.2"/>
-  <joint name="gripper_base_joint" type="fixed">
-    <parent link="end_effector"/>
-    <child link="gripper_base"/>
-    <origin xyz="0 0 0.02" rpy="0 0 0"/>
-  </joint>
-  <xacro:box_link name="gripper_base" size="0.08 0.06 0.02" xyz="0 0 0" rpy="0 0 0" color="0.5 0.5 0.5 1.0" mass="0.2"/>
-  <!-- Left finger -->
-  <joint name="left_finger_joint" type="prismatic">
-    <parent link="gripper_base"/>
-    <child link="left_finger"/>
-    <origin xyz="0.04 0.02 0.01" rpy="0 0 0"/>
-    <axis xyz="0 1 0"/>
-    <limit lower="0.0" upper="0.03" effort="50.0" velocity="0.5"/>
-    <dynamics damping="0.1" friction="0.05"/>
-  </joint>
-  <xacro:box_link name="left_finger" size="0.03 0.01 0.06" xyz="0 0 0.03" rpy="0 0 0" color="1.0 0.5 0.0 1.0" mass="0.05"/>
-  <!-- Right finger -->
-  <joint name="right_finger_joint" type="prismatic">
-    <parent link="gripper_base"/>
-    <child link="right_finger"/>
-    <origin xyz="0.04 -0.02 0.01" rpy="0 0 0"/>
-    <axis xyz="0 -1 0"/>
-    <limit lower="0.0" upper="0.03" effort="50.0" velocity="0.5"/>
-    <dynamics damping="0.1" friction="0.05"/>
-    <mimic joint="left_finger_joint" multiplier="1" offset="0"/>
-  </joint>
-  <xacro:box_link name="right_finger" size="0.03 0.01 0.06" xyz="0 0 0.03" rpy="0 0 0" color="1.0 0.5 0.0 1.0" mass="0.05"/>
-  <!-- ROS2 Control Hardware Interface -->
-  <ros2_control name="GazeboSystem" type="system">
-    <hardware>
-      <plugin name="gazebo_ros2_control/GazeboSystem"/>
-    </hardware>
-    <joint name="shoulder_yaw_joint">
-      <command_interface name="position"/>
-      <state_interface name="position"/>
-      <state_interface name="velocity"/>
-      <state_interface name="effort"/>
-    </joint>
-    <joint name="shoulder_pitch_joint">
-      <command_interface name="position"/>
-      <state_interface name="position"/>
-      <state_interface name="velocity"/>
-      <state_interface name="effort"/>
-    </joint>
-    <joint name="elbow_joint">
-      <command_interface name="position"/>
-      <state_interface name="position"/>
-      <state_interface name="velocity"/>
-      <state_interface name="effort"/>
-    </joint>
-    <joint name="wrist_roll_joint">
-      <command_interface name="position"/>
-      <state_interface name="position"/>
-      <state_interface name="velocity"/>
-      <state_interface name="effort"/>
-    </joint>
-    <joint name="wrist_pitch_joint">
-      <command_interface name="position"/>
-      <state_interface name="position"/>
-      <state_interface name="velocity"/>
-      <state_interface name="effort"/>
-    </joint>
-    <joint name="left_finger_joint">
-      <command_interface name="position"/>
-      <state_interface name="position"/>
-      <state_interface name="velocity"/>
-      <state_interface name="effort"/>
-    </joint>
-    <joint name="right_finger_joint">
-      <command_interface name="position"/>
-      <state_interface name="position"/>
-      <state_interface name="velocity"/>
-      <state_interface name="effort"/>
-    </joint>
-  </ros2_control>
-</robot>
+/home/aniketh05/ros2_ws/src/my_gesture_arm/model/my_gesture_arm.xacro
